File: hardware/esp32-cam-hw.kicad_sch (KiCad schematic)
At the start: 10 parts, among them J2 Conn_01x05_Pin, J3 Conn_01x04_Pin, J4 Conn_01x04_Pin, SW1 SW_Push, U2 Micro_USB_Converter

Commit message: Hardware: Center front panel components and add custom switch footprint
- Centered front panel components (SW1, D1, D2, J3, J4) precisely on the X-axis for optical symmetry.
- Added a custom KiCad footprint for the DTR 7/RT push button (9.5mm body, round).
- Adjusted THT pad sizes for the custom switch (2.6mm outer diameter, 2.0mm drill) to guarantee a minimum 0.6mm gap for CNC isolation milling.
- Updated README.md to reflect the specific switch model and adjusted PCB milling specifications.
Parts:
- SW1: footprint Connector_PinHeader_2.54mm:PinHeader_1x02_P2.54mm_Vertical -> FootprintLibrary:SW_DTR_7_RT
Changed lines of the file:
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@@
 			)
 		)
-		(property "Footprint" "Connector_PinHeader_2.54mm:PinHeader_1x02_P2.54mm_Vertical"
+		(property "Footprint" "FootprintLibrary:SW_DTR_7_RT"
 			(at 227.33 34.29 0)
 			(effects
